File: pcb/karl/karl.kicad_pcb (KiCad board)
At the start: 2 copper layers, 76.2 x 41.9 mm, 8 parts, among them J1 Raspberry_Pi, J2 Power, J3 Battery, J4 LIDAR_Power, J5 Motor_Power, U1 MCP3421A0T-ECH

Commit message: added turning lights
Parts:
- added D1: RED, LED_SMD:LED_0603_1608Metric, F.Cu at (47.0, 38.9)
- added D2: Orange, LED_SMD:LED_0603_1608Metric, F.Cu at (95.2, 63.5)
- added D3: Orange, LED_SMD:LED_0603_1608Metric, F.Cu at (30.5, 67.3)
- added D4: Orange, LED_SMD:LED_0603_1608Metric, F.Cu at (95.2, 67.3)
- added D5: Orange, LED_SMD:LED_0603_1608Metric, F.Cu at (30.5, 63.5)
- added D6: Orange, LED_SMD:LED_0603_1608Metric, F.Cu at (95.2, 22.9)
- added D7: Orange, LED_SMD:LED_0603_1608Metric, F.Cu at (30.5, 26.7)
- added D8: Orange, LED_SMD:LED_0603_1608Metric, F.Cu at (95.2, 26.7)
- added D9: Orange, LED_SMD:LED_0603_1608Metric, F.Cu at (30.5, 22.9)
- added Q1: MMBT3904, Package_TO_SOT_SMD:SOT-23, F.Cu at (45.4, 61.2)
- added Q2: MMBT3904, Package_TO_SOT_SMD:SOT-23, F.Cu at (50.5, 61.2)
- added R10: 100R, Resistor_SMD:R_0603_1608Metric, F.Cu at (91.4, 22.9)
- added R11: 100R, Resistor_SMD:R_0603_1608Metric, F.Cu at (34.3, 26.7)
- added R12: 100R, Resistor_SMD:R_0603_1608Metric, F.Cu at (91.4, 26.7)
- added R13: 100R, Resistor_SMD:R_0603_1608Metric, F.Cu at (34.3, 22.9)
- added R3: 5k6, Resistor_SMD:R_0603_1608Metric, F.Cu at (43.7, 64.8)
- added R4: 5k6, Resistor_SMD:R_0603_1608Metric, F.Cu at (48.7, 64.8)
- added R5: 120R, Resistor_SMD:R_0603_1608Metric, F.Cu at (49.5, 38.9)
- added R6: 100R, Resistor_SMD:R_0603_1608Metric, F.Cu at (91.4, 63.5)
- added R7: 100R, Resistor_SMD:R_0603_1608Metric, F.Cu at (34.3, 67.3)
- added R8: 100R, Resistor_SMD:R_0603_1608Metric, F.Cu at (91.4, 67.3)
- added R9: 100R, Resistor_SMD:R_0603_1608Metric, F.Cu at (34.3, 63.5)
- moved J1 12.7 mm to (39.4, 74.9)
Connections:
- J1 pad 16: Net-(J1-Pad16) -> GPIO_23
- J1 pad 18: Net-(J1-Pad18) -> GPIO_24
Routing:
- net +5V: track 68.4 -> 206.6 mm
- net Net-(D2-Pad1): track 0.00 -> 104.4 mm, vias 0 -> 2
- net Net-(D3-Pad1): track 0.00 -> 69.0 mm, vias 0 -> 3
- net +3V3: track 22.4 -> 0.00 mm
- net GPIO_23: track 0.00 -> 20.2 mm
- net GND: track 103.2 -> 122.9 mm, vias 0 -> 4
- net GPIO_24: track 0.00 -> 17.4 mm
- net SCL: track 43.4 -> 26.7 mm
- net SDA: track 40.1 -> 29.9 mm
- net Net-(Q2-Pad1): track 0.00 -> 2.54 mm
- net Net-(Q1-Pad1): track 0.00 -> 2.54 mm
- net Net-(D1-Pad2): track 0.00 -> 2.54 mm
- net Net-(D9-Pad2): track 0.00 -> 2.23 mm
- net Net-(D8-Pad2): track 0.00 -> 2.23 mm
- net Net-(D7-Pad2): track 0.00 -> 2.23 mm
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Other:
- board size 76.2 x 41.9 mm -> 72.4 x 57.1 mm
- board text removed: "V_1.0"

Commit message: minor changes
Other:
- board text added: "1"
- board text added: "40"
Changed lines of the file:
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@@
   (general
     (thickness 1.6)
-    (drawings 16)
+    (drawings 18)
     (tracks 197)
     (zones 0)
@@
     )
   )
+  (gr_text "40\n" (at 90.17 71.12) (layer F.SilkS)
+    (effects (font (size 1 1) (thickness 0.2)))
+  )
+  (gr_text 1 (at 36.83 76.2) (layer F.SilkS)
+    (effects (font (size 1 1) (thickness 0.2)))
+  )
   (gr_line (start 99.06 77.47) (end 99.06 76.2) (layer Edge.Cuts) (width 0.05))

Commit message: saved
Other:
- board text removed: "-KARL-"
Changed lines of the file:
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@@
   (general
     (thickness 1.6)
-    (drawings 18)
+    (drawings 17)
     (tracks 197)
     (zones 0)
@@
     (effects (font (size 1.5 1.5) (thickness 0.3)) (justify left))
   )
-  (gr_text "-KARL-\n " (at 76.2 44.45 180) (layer F.Cu)
-    (effects (font (size 5 5) (thickness 0.6)))
-  )
   (gr_text "c Manuel Fehren" (at 73.66 21.59 180) (layer F.SilkS)
